Commit message: Added Gazebo simulation

File: iiwa_description/urdf/iiwa.transmission.xacro (robot description, xacro)
@@ -2,77 +2,77 @@
 <robot xmlns:xacro="http://www.ros.org/wiki/xacro">
   <xacro:macro name="iiwa_transmission" params="hardware_interface">
-    <transmission name="${robot_name}_tran_1">
+    <transmission name="tran_1">
       <robotNamespace>/${robot_name}</robotNamespace>
       <type>transmission_interface/SimpleTransmission</type>
-      <joint name="${robot_name}_joint_1">
+      <joint name="joint_1">
 	<hardwareInterface>${hardware_interface}</hardwareInterface>
       </joint>
-      <actuator name="${robot_name}_motor_1">
+      <actuator name="motor_1">
 	<hardwareInterface>${hardware_interface}</hardwareInterface>
 	<mechanicalReduction>1</mechanicalReduction>
       </actuator>
     </transmission>
-    <transmission name="${robot_name}_tran_2">
+    <transmission name="tran_2">
       <robotNamespace>/${robot_name}</robotNamespace>
       <type>transmission_interface/SimpleTransmission</type>
-      <joint name="${robot_name}_joint_2">
+      <joint name="joint_2">
 	<hardwareInterface>${hardware_interface}</hardwareInterface>
       </joint>
-      <actuator name="${robot_name}_motor_2">
+      <actuator name="motor_2">
 	<hardwareInterface>${hardware_interface}</hardwareInterface>
 	<mechanicalReduction>1</mechanicalReduction>
       </actuator>
     </transmission>
-    <transmission name="${robot_name}_tran_3">
+    <transmission name="tran_3">
       <robotNamespace>/${robot_name}</robotNamespace>
       <type>transmission_interface/SimpleTransmission</type>
-      <joint name="${robot_name}_joint_3">
+      <joint name="joint_3">
 	<hardwareInterface>${hardware_interface}</hardwareInterface>
       </joint>
-      <actuator name="${robot_name}_motor_3">
+      <actuator name="motor_3">
 	<hardwareInterface>${hardware_interface}</hardwareInterface>
 	<mechanicalReduction>1</mechanicalReduction>
       </actuator>
     </transmission>
-    <transmission name="${robot_name}_tran_4">
+    <transmission name="tran_4">
       <robotNamespace>/${robot_name}</robotNamespace>
       <type>transmission_interface/SimpleTransmission</type>
-      <joint name="${robot_name}_joint_4">
+      <joint name="joint_4">
 	<hardwareInterface>${hardware_interface}</hardwareInterface>
       </joint>
-      <actuator name="${robot_name}_motor_4">
+      <actuator name="motor_4">
 	<hardwareInterface>${hardware_interface}</hardwareInterface>
 	<mechanicalReduction>1</mechanicalReduction>
       </actuator>
     </transmission>
-    <transmission name="${robot_name}_tran_5">
+    <transmission name="tran_5">
       <robotNamespace>/${robot_name}</robotNamespace>
       <type>transmission_interface/SimpleTransmission</type>
-      <joint name="${robot_name}_joint_5">
+      <joint name="joint_5">
 	<hardwareInterface>${hardware_interface}</hardwareInterface>
       </joint>
-      <actuator name="${robot_name}_motor_5">
+      <actuator name="motor_5">
 	<hardwareInterface>${hardware_interface}</hardwareInterface>
 	<mechanicalReduction>1</mechanicalReduction>
       </actuator>
     </transmission>
-    <transmission name="${robot_name}_tran_6">
+    <transmission name="tran_6">
       <robotNamespace>/${robot_name}</robotNamespace>
       <type>transmission_interface/SimpleTransmission</type>
-      <joint name="${robot_name}_joint_6">
+      <joint name="joint_6">
 	<hardwareInterface>${hardware_interface}</hardwareInterface>
       </joint>
-      <actuator name="${robot_name}_motor_6">
+      <actuator name="motor_6">
 	<hardwareInterface>${hardware_interface}</hardwareInterface>
 	<mechanicalReduction>1</mechanicalReduction>
       </actuator>
     </transmission>
-    <transmission name="${robot_name}_tran_7">
+    <transmission name="tran_7">
       <robotNamespace>/${robot_name}</robotNamespace>
       <type>transmission_interface/SimpleTransmission</type>
-      <joint name="${robot_name}_joint_7">
+      <joint name="joint_7">
 	<hardwareInterface>${hardware_interface}</hardwareInterface>
       </joint>
-      <actuator name="${robot_name}_motor_7">
+      <actuator name="motor_7">
 	<hardwareInterface>${hardware_interface}</hardwareInterface>
 	<mechanicalReduction>1</mechanicalReduction>

File: iiwa_description/urdf/iiwa14.xacro (robot description, xacro)
@@ -63,5 +63,5 @@
     </link>
     <!-- joint between link_0 and link_1 -->
-    <joint name="joint_0" type="revolute">
+    <joint name="joint_1" type="revolute">
       <parent link="link_0"/>
       <child link="link_1"/>
@@ -98,5 +98,5 @@
     </link>
     <!-- joint between link_1 and link_2 -->
-    <joint name="joint_1" type="revolute">
+    <joint name="joint_2" type="revolute">
       <parent link="link_1"/>
       <child link="link_2"/>
@@ -133,5 +133,5 @@
     </link>
     <!-- joint between link_2 and link_3 -->
-    <joint name="joint_2" type="revolute">
+    <joint name="joint_3" type="revolute">
       <parent link="link_2"/>
       <child link="link_3"/>
@@ -168,5 +168,5 @@
     </link>
    <!-- joint between link_3 and link_4 -->
-    <joint name="joint_3" type="revolute">
+    <joint name="joint_4" type="revolute">
       <parent link="link_3"/>
       <child link="link_4"/>
@@ -203,5 +203,5 @@
     </link>
     <!-- joint between link_4 and link_5 -->
-    <joint name="joint_4" type="revolute">
+    <joint name="joint_5" type="revolute">
       <parent link="link_4"/>
       <child link="link_5"/>
@@ -238,5 +238,5 @@
     </link>
  <!-- joint between link_5 and link_6 -->
-    <joint name="joint_5" type="revolute">
+    <joint name="joint_6" type="revolute">
       <parent link="link_5"/>
       <child link="link_6"/>
@@ -273,5 +273,5 @@
     </link>
  <!-- joint between link_6 and link_7 -->
-    <joint name="joint_6" type="revolute">
+    <joint name="joint_7" type="revolute">
       <parent link="link_6"/>
       <child link="link_7"/>

File: iiwa_description/urdf/iiwa7.xacro (robot description, xacro)
@@ -15,10 +15,10 @@
   <xacro:macro name="iiwa7" params="parent hardware_interface robot_name *origin">
     <!--joint between {parent} and link_0-->
-    <joint name="${parent}_${robot_name}_joint" type="fixed">
+    <joint name="${parent}_joint" type="fixed">
       <xacro:insert_block name="origin"/>
       <parent link="${parent}"/>
-      <child link="${robot_name}_link_0"/>
-    </joint>
-    <link name="${robot_name}_link_0">
+      <child link="link_0"/>
+    </joint>
+    <link name="link_0">
       <inertial>
         <origin xyz="-0.1 0 0.07" rpy="0 0 0"/>
@@ -48,7 +48,7 @@
     </link>
     <!-- joint between link_0 and link_1 -->
-    <joint name="${robot_name}_joint_1" type="revolute">
-      <parent link="${robot_name}_link_0"/>
-      <child link="${robot_name}_link_1"/>
+    <joint name="joint_1" type="revolute">
+      <parent link="link_0"/>
+      <child link="link_1"/>
       <origin xyz="0 0 0.15" rpy="0 0 0"/>
       <axis xyz="0 0 1"/>
@@ -61,5 +61,5 @@
       <dynamics damping="${joint_damping}"/>
     </joint>
-    <link name="${robot_name}_link_1">
+    <link name="link_1">
       <inertial>
         <origin xyz="0 -0.03 0.12" rpy="0 0 0"/>
@@ -82,7 +82,7 @@
       </collision>
     </link>
-    <joint name="${robot_name}_joint_2" type="revolute">
-      <parent link="${robot_name}_link_1"/>
-      <child link="${robot_name}_link_2"/>
+    <joint name="joint_2" type="revolute">
+      <parent link="link_1"/>
+      <child link="link_2"/>
       <origin xyz="0 0 0.19" rpy="${PI / 2}   0 ${PI}"/>
       <axis xyz="0 0 1"/>
@@ -95,5 +95,5 @@
       <dynamics damping="${joint_damping}"/>
     </joint>
-    <link name="${robot_name}_link_2">
+    <link name="link_2">
       <inertial>
         <origin xyz="0.0003 0.059 0.042" rpy="0 0 0"/>
@@ -116,7 +116,7 @@
       </collision>
     </link>
-    <joint name="${robot_name}_joint_3" type="revolute">
-      <parent link="${robot_name}_link_2"/>
-      <child link="${robot_name}_link_3"/>
+    <joint name="joint_3" type="revolute">
+      <parent link="link_2"/>
+      <child link="link_3"/>
       <origin xyz="0 0.21 0" rpy="${PI / 2} 0 ${PI}"/>
       <axis xyz="0 0 1"/>
@@ -129,5 +129,5 @@
       <dynamics damping="${joint_damping}"/>
     </joint>
-    <link name="${robot_name}_link_3">
+    <link name="link_3">
       <inertial>
         <origin xyz="0 0.03 0.13" rpy="0 0 0"/>
@@ -150,7 +150,7 @@
       </collision>
     </link>
-    <joint name="${robot_name}_joint_4" type="revolute">
-      <parent link="${robot_name}_link_3"/>
-      <child link="${robot_name}_link_4"/>
+    <joint name="joint_4" type="revolute">
+      <parent link="link_3"/>
+      <child link="link_4"/>
       <origin xyz="0 0 0.19" rpy="${PI / 2} 0 0"/>
       <axis xyz="0 0 1"/>
@@ -163,5 +163,5 @@
       <dynamics damping="${joint_damping}"/>
     </joint>
-    <link name="${robot_name}_link_4">
+    <link name="link_4">
       <inertial>
         <origin xyz="0 0.067 0.034" rpy="0 0 0"/>
@@ -184,7 +184,7 @@
       </collision>
     </link>
-    <joint name="${robot_name}_joint_5" type="revolute">
-      <parent link="${robot_name}_link_4"/>
-      <child link="${robot_name}_link_5"/>
+    <joint name="joint_5" type="revolute">
+      <parent link="link_4"/>
+      <child link="link_5"/>
       <origin xyz="0 0.21 0" rpy="${-PI / 2} ${PI} 0"/>
       <axis xyz="0 0 1"/>
@@ -197,5 +197,5 @@
       <dynamics damping="${joint_damping}"/>
     </joint>
-    <link name="${robot_name}_link_5">
+    <link name="link_5">
       <inertial>
         <origin xyz="0.0001 0.021 0.076" rpy="0 0 0"/>
@@ -218,7 +218,7 @@
       </collision>
     </link>
-    <joint name="${robot_name}_joint_6" type="revolute">
-      <parent link="${robot_name}_link_5"/>
-      <child link="${robot_name}_link_6"/>
+    <joint name="joint_6" type="revolute">
+      <parent link="link_5"/>
+      <child link="link_6"/>
       <origin xyz="0 0.06070 0.19" rpy="${PI / 2} 0 0"/>
       <axis xyz="0 0 1"/>
@@ -231,5 +231,5 @@
       <dynamics damping="${joint_damping}"/>
     </joint>
-    <link name="${robot_name}_link_6">
+    <link name="link_6">
       <inertial>
         <origin xyz="0 0.0006 0.0004" rpy="0 0 0"/>
@@ -252,7 +252,7 @@
       </collision>
     </link>
-    <joint name="${robot_name}_joint_7" type="revolute">
-      <parent link="${robot_name}_link_6"/>
-      <child link="${robot_name}_link_7"/>
+    <joint name="joint_7" type="revolute">
+      <parent link="link_6"/>
+      <child link="link_7"/>
       <origin xyz="0 0.081 0.06070" rpy="${- PI / 2} ${PI} 0"/>
       <axis xyz="0 0 1"/>
@@ -265,5 +265,5 @@
       <dynamics damping="${joint_damping}"/>
     </joint>
-    <link name="${robot_name}_link_7">
+    <link name="link_7">
       <inertial>
         <origin xyz="0 0 0.02" rpy="0 0 0"/>
@@ -286,10 +286,10 @@
       </collision>
     </link>
-    <joint name="${robot_name}_joint_ee" type="fixed">
-      <parent link="${robot_name}_link_7"/>
-      <child link="${robot_name}_link_ee"/>
+    <joint name="joint_ee" type="fixed">
+      <parent link="link_7"/>
+      <child link="link_ee"/>
       <origin xyz="0 0 0.045" rpy="0 0 0"/>
     </joint>
-    <link name="${robot_name}_link_ee">
+    <link name="link_ee">
       <inertial>
         <origin xyz="0 0 0" rpy="0 0 0"/>
